File: hardware/PicoLink.kicad_pcb (KiCad board)
At the start: 2 copper layers, 56.1 x 38.2 mm, 50 parts, among them J2 USB_C_Receptacle_USB2.0_14P, J3 ARM_JTAG_10Pin, J4 TARGET, J7 UART, J8 SIGROK_INPUT, J9 SIGROK_ADC, SW2 BOOT SELECTOR, U4 W25Q16JVSS, U6 AMS1117-3.3, Y2 12Mhz HC49-SD

Commit message: [07-20-0908] update gerber and schematic
Parts:
- removed C19, C21, C22, C27, C28, C29, C30, C31, C32: 100nF, Capacitor_SMD:C_0603_1608Metric_Pad1.08x0.95mm_HandSolder
- removed C20, C26: 2u2F, Capacitor_SMD:C_0603_1608Metric_Pad1.08x0.95mm_HandSolder
- removed C23: 12pF, Capacitor_SMD:C_0603_1608Metric_Pad1.08x0.95mm_HandSolder
- removed D2: green, LED_SMD:LED_0805_2012Metric_Pad1.15x1.40mm_HandSolder
- removed J8: SIGROK_INPUT, Connector_PinHeader_2.54mm:PinHeader_1x07_P2.54mm_Vertical
- removed J9: SIGROK_ADC, Connector_PinHeader_2.54mm:PinHeader_1x03_P2.54mm_Vertical
- removed R21: 1K, Resistor_SMD:R_0805_2012Metric_Pad1.20x1.40mm_HandSolder
- removed RP1: RP2040, Package_DFN_QFN:QFN-56-1EP_7x7mm_P0.4mm_EP3.2x3.2mm
- removed Y2: 12Mhz HC49-SD, Crystal:Crystal_SMD_HC49-SD_HandSoldering
- added C10: 100nF, Capacitor_SMD:C_0603_1608Metric_Pad1.08x0.95mm_HandSolder, F.Cu at (170.9, 85.6)
- added C11: 100nF, Capacitor_SMD:C_0603_1608Metric_Pad1.08x0.95mm_HandSolder, F.Cu at (169.2, 85.6)
- added C12: 100nF, Capacitor_SMD:C_0603_1608Metric_Pad1.08x0.95mm_HandSolder, F.Cu at (167.6, 85.6)
- added C13: 12pF, Capacitor_SMD:C_0603_1608Metric_Pad1.08x0.95mm_HandSolder, F.Cu at (162.7, 102.2)
- added C2: 2u2F, Capacitor_SMD:C_0603_1608Metric_Pad1.08x0.95mm_HandSolder, F.Cu at (159.1, 85.6)
- added C3: 100nF, Capacitor_SMD:C_0603_1608Metric_Pad1.08x0.95mm_HandSolder, F.Cu at (162.5, 85.6)
- added C4: 100nF, Capacitor_SMD:C_0603_1608Metric_Pad1.08x0.95mm_HandSolder, F.Cu at (160.8, 85.6)
- added C5: 1uF, Capacitor_SMD:C_0603_1608Metric_Pad1.08x0.95mm_HandSolder, F.Cu at (166.3, 103.3)
- added C6: 100nF, Capacitor_SMD:C_0603_1608Metric_Pad1.08x0.95mm_HandSolder, F.Cu at (168.0, 103.3)
- added C7: 100nF, Capacitor_SMD:C_0603_1608Metric_Pad1.08x0.95mm_HandSolder, F.Cu at (169.7, 103.3)
- added C8: 100nF, Capacitor_SMD:C_0603_1608Metric_Pad1.08x0.95mm_HandSolder, F.Cu at (165.8, 85.6)
- added C9: 100nF, Capacitor_SMD:C_0603_1608Metric_Pad1.08x0.95mm_HandSolder, F.Cu at (164.2, 85.6)
- added D1: green, LED_SMD:LED_0805_2012Metric_Pad1.15x1.40mm_HandSolder, F.Cu at (167.8, 97.5)
- added J1: SIGROK_ADC, Connector_PinHeader_2.54mm:PinHeader_1x03_P2.54mm_Vertical, B.Cu at (163.1, 97.0)
- added J5: SIGROK_INPUT, Connector_PinHeader_2.54mm:PinHeader_1x07_P2.54mm_Vertical, B.Cu at (148.4, 107.8)
- added R2: 1K, Resistor_SMD:R_0805_2012Metric_Pad1.20x1.40mm_HandSolder, F.Cu at (164.6, 102.1)
- added R3: 1K, Resistor_SMD:R_0805_2012Metric_Pad1.20x1.40mm_HandSolder, F.Cu at (167.8, 99.7)
- added U1: RP2040, Package_DFN_QFN:QFN-56-1EP_7x7mm_P0.4mm_EP3.2x3.2mm, F.Cu at (155.7, 92.7)
- added Y1: 12Mhz HC49-SD, Crystal:Crystal_SMD_HC49-SD, F.Cu at (152.8, 102.5)
- moved C1 5.91 mm to (161.0, 102.2), turned to -90 degrees
- moved R23 0.47 mm to (147.7, 89.7)
- moved R24 0.47 mm to (147.7, 91.8)
- moved R25 0.47 mm to (147.7, 93.8)
- moved R26 0.47 mm to (147.7, 95.9)
Routing:
- net Net-(RP1-VREG_VOUT): track 34.0 -> 0.00 mm
- net +1V1: track 0.00 -> 33.3 mm
- net Net-(D2-A): track 13.8 -> 0.00 mm
- net Net-(D1-A): track 0.00 -> 13.8 mm
- net Net-(C13-Pad1): track 0.00 -> 11.9 mm
- net /XIN: track 12.9 -> 19.8 mm
- net +3.3V: track 142.2 -> 147.8 mm
- net GND: track 250.8 -> 253.1 mm
- net Net-(D2-K): track 2.11 -> 0.00 mm
- net Net-(D1-K): track 0.00 -> 2.11 mm
- net SWD_CLK: track 0.00 -> 1.96 mm
- net /XOUT: track 11.7 -> 13.5 mm
- net unconnected-(U1-GPIO0-Pad2): track 0.00 -> 1.46 mm
- net unconnected-(RP1-GPIO0-Pad2): track 1.46 -> 0.00 mm
- net /SIGROK_IN6: track 32.4 -> 33.7 mm
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- added copper zone on B.Cu, net +3.3V
